File: Hardware/MLX90393_Magnetometer_Breakout.sch (EAGLE design)
At the start: 16 parts, among them U1 MLX90393_MAGNETOMETER

Commit message: Adding bottom silk
Other:
- note added: "Default 7-bit I2C Adr: 0x0C"
Changed lines of the file:
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@@
   SJ1 must be open for SPI operation.</text>
 <text x="205.994" y="133.35" size="1.778" layer="97">I2C Addressing Table</text>
+<text x="199.898" y="81.788" size="1.778" layer="97">Default 7-bit I2C Adr: 0x0C</text>
 </plain>
 <instances>
