File: Hardware/MLX90393_Magnetometer_Breakout.sch (EAGLE design)
At the start: 15 parts, among them U1 MLX90393_MAGNETOMETER

Commit message: Bringing back production layout: missing top mask on QFN.
Parts:
- added U$1: OSHW-LOGOS, SparkFun:OSHW-LOGOS
Connections:
- net VDD renamed 3.3V
- net INT: now also J1.5
- net TRIG: now also J1.6
Other:
- note added: "Address selection jumpers"
- note added: "Default 7-bit I2C Adr: 0x0C"
- note added: "I2C Port"
- note added: "SJ1 Controls I2C/SPI Closed (Default): I2C Open: SPI"
- note added: "SPI Port"
- note added: "VCC must be 2.2-3.6V"
- note removed: "Address selection jumpers SJ3 and SJ4"
- note removed: "Apply regulated 2.2-3.6V to VDD"
- note removed: "I2C Ports"
- note removed: "Pulling up SENB/CS to VDD through SJ1 enables I2C mode."
- note removed: "SPI Ports"
- moved on the sheet: C1, C4
